File: pic_programmer/pic_programmer.sch (KiCad schematic (older format))
At the start: 56 parts, among them J1 DB9-FEMAL, P1 CONN_2, P101 CONN_1, P102 CONN_1, P103 CONN_1, P104 CONN_1, P105 CONN_1, P106 CONN_1, Q1 BC237, Q2 BC307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

Commit message: add more and modify
Other:
- note added: "Try to change in Sch\n"
- note removed: "!@#$!@#$153154\n"
Changed lines of the file:
@@
 NoConn ~ 6250 7400
 NoConn ~ 6250 7550
-Text Notes 8300 1150 0    197  ~ 0
-!@#$!@#$153154\n
+Text Notes 7400 1000 0    197  ~ 0
+Try to change in Sch\n
 $EndSCHEMATC

Commit message: change in sch
Other:
- note added: "3rd Change"
- note removed: "Try to change in Sch\n"
Changed lines of the file:
@@
 NoConn ~ 6250 7550
 Text Notes 7400 1000 0    197  ~ 0
-Try to change in Sch\n
+3rd Change
 $EndSCHEMATC
